Commit message: adapted ycb sampling

File: assets/xacro/generic_ycb_exploration.xml.xacro (robot description, xacro)
@@ -26,4 +26,5 @@
         <material name="object_material" specular="0" shininess="0.5" reflectance="0" rgba="0.3 0.3 0.8 0.8" />
         <material name="glance_material" specular="0" shininess="0.5" reflectance="0" rgba="0 1 0 0.13" />
+        <material name="alignment_material" specular="0" shininess="0.5" reflectance="0" rgba="1 0 0 0.13" />
 	</asset>
     <xacro:object_asset object_model_subpath="$(arg mesh_subpath)"/>
@@ -32,4 +33,6 @@
 		<geom name="table" pos="0 0 0.18" size="0.2 0.2 0.18" type="box" material="table_material"/>
 		<site name="glance_site" pos="0 0 0.39" type="box" material="glance_material" size="0.18 0.14 0.12"/>
+		<site name="align1" pos="0 0 0.39" type="box" material="alignment_material" size="0.2 0.002 0.12"/>
+		<site name="align2" pos="0 0 0.39" type="box" material="alignment_material" size="0.002 0.2 0.12"/>
 		<body name="board_boundary" pos="0 0 0.36">
 			<geom type="box" pos="0.125 0 0.015" size="0.075 0.2 0.015"/>

Commit message: Adds object rotation

File: assets/xacro/generic_ycb_exploration.xml.xacro (robot description, xacro)
@@ -6,4 +6,5 @@
     <xacro:arg name="mesh_pos" default="0 0 0" />
     <xacro:arg name="mesh_rot" default="0 0 0" />
+    <xacro:arg name="mesh_theta" default="0" />
     <xacro:arg name="use_panda" default="0" />
     <xacro:include filename="$(find haptic_exploration)/assets/xacro/object.xml.xacro" />
@@ -54,5 +55,5 @@
 		<light directional="true" ambient="0.2 0.2 0.2" diffuse="0.8 0.8 0.8" specular="0.3 0.3 0.3" castshadow="false" pos="0 0 4" dir="0 0 -1" name="light0" />
 		<xacro:if value="$(arg use_object)" >
-			<xacro:object_body pos="$(arg mesh_pos)" rot="$(arg mesh_rot)"/>
+			<xacro:object_body pos="$(arg mesh_pos)" rot="$(arg mesh_rot)" theta="$(arg mesh_theta)"/>
 		</xacro:if>
 	</worldbody>

File: assets/xacro/object.xml.xacro (robot description, xacro)
@@ -6,6 +6,6 @@
         </asset>
     </xacro:macro>
-    <xacro:macro name="object_body" params="pos rot">
-        <body name="object" pos="0 0.0 0.36" >
+    <xacro:macro name="object_body" params="pos rot theta">
+        <body name="object" pos="0 0.0 0.36" euler="0 0 ${theta}">
             <!-- <freejoint /> -->
             <geom name="object_geom" type="mesh" mesh="object_collision" pos="${pos}" euler="${rot}" material="object_material" rgba="0.3 0.3 0.8 0.8" group="1" contype="2" conaffinity="1" />
